File: Guitutar_LEDS.sch (EAGLE design)
At the start: 161 parts

Commit message: Created new schematic of just the stamp board and made layout for the schematic.
Connections:
- new net N$165: U$6.SER
Changed lines of the file:
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@@
 <wire x1="274.32" y1="167.64" x2="274.32" y2="127" width="0.1524" layer="91"/>
 <wire x1="274.32" y1="251.46" x2="274.32" y2="208.28" width="0.1524" layer="91"/>
+<wire x1="274.32" y1="58.42" x2="302.26" y2="58.42" width="0.1524" layer="91"/>
+<label x="302.26" y="58.42" size="1.27" layer="95" xref="yes"/>
 </segment>
 </net>
@@
 <wire x1="269.24" y1="162.56" x2="269.24" y2="121.92" width="0.1524" layer="91"/>
 <wire x1="269.24" y1="246.38" x2="269.24" y2="203.2" width="0.1524" layer="91"/>
+<wire x1="269.24" y1="53.34" x2="292.1" y2="53.34" width="0.1524" layer="91"/>
+<label x="292.1" y="53.34" size="1.27" layer="95" xref="yes"/>
 </segment>
 </net>
@@
 <wire x1="266.7" y1="160.02" x2="266.7" y2="119.38" width="0.1524" layer="91"/>
 <wire x1="266.7" y1="243.84" x2="266.7" y2="200.66" width="0.1524" layer="91"/>
+<wire x1="266.7" y1="50.8" x2="287.02" y2="50.8" width="0.1524" layer="91"/>
+<label x="287.02" y="50.8" size="1.27" layer="95" xref="yes"/>
 </segment>
 </net>
@@
 <wire x1="271.78" y1="248.92" x2="271.78" y2="205.74" width="0.1524" layer="91"/>
 <wire x1="182.88" y1="83.82" x2="182.88" y2="55.88" width="0.1524" layer="91"/>
+<wire x1="271.78" y1="55.88" x2="297.18" y2="55.88" width="0.1524" layer="91"/>
+<label x="297.18" y="55.88" size="1.27" layer="95" xref="yes"/>
 </segment>
 </net>
@@
 <pinref part="U$1" gate="G$1" pin="SER"/>
 <wire x1="76.2" y1="375.92" x2="106.68" y2="375.92" width="0.1524" layer="91"/>
+<label x="106.68" y="375.92" size="1.27" layer="95" xref="yes"/>
 </segment>
 </net>
@@
 <pinref part="U$2" gate="G$1" pin="SER"/>
 <wire x1="76.2" y1="335.28" x2="106.68" y2="335.28" width="0.1524" layer="91"/>
+<label x="106.68" y="335.28" size="1.27" layer="95" xref="yes"/>
 </segment>
 </net>
@@
 <pinref part="U$3" gate="G$1" pin="SER"/>
 <wire x1="76.2" y1="294.64" x2="106.68" y2="294.64" width="0.1524" layer="91"/>
+<label x="106.68" y="294.64" size="1.27" layer="95" xref="yes"/>
 </segment>
 </net>
@@
 <pinref part="U$4" gate="G$1" pin="SER"/>
 <wire x1="76.2" y1="254" x2="106.68" y2="254" width="0.1524" layer="91"/>
+<label x="106.68" y="254" size="1.27" layer="95" xref="yes"/>
 </segment>
 </net>
@@
 <pinref part="U$5" gate="G$1" pin="SER"/>
 <wire x1="76.2" y1="210.82" x2="106.68" y2="210.82" width="0.1524" layer="91"/>
+<label x="106.68" y="210.82" size="1.27" layer="95" xref="yes"/>
 </segment>
 </net>
@@
 <pinref part="U$7" gate="G$1" pin="SER"/>
 <wire x1="76.2" y1="129.54" x2="109.22" y2="129.54" width="0.1524" layer="91"/>
+<label x="109.22" y="129.54" size="1.27" layer="95" xref="yes"/>
 </segment>
 </net>
@@
 <pinref part="U$8" gate="G$1" pin="SER"/>
 <wire x1="76.2" y1="88.9" x2="106.68" y2="88.9" width="0.1524" layer="91"/>
+<label x="106.68" y="88.9" size="1.27" layer="95" xref="yes"/>
 </segment>
 </net>
@@
 <pinref part="U$16" gate="G$1" pin="SER"/>
 <wire x1="165.1" y1="88.9" x2="195.58" y2="88.9" width="0.1524" layer="91"/>
+<label x="195.58" y="88.9" size="1.27" layer="95" xref="yes"/>
 </segment>
 </net>
@@
 <pinref part="U$15" gate="G$1" pin="SER"/>
 <wire x1="165.1" y1="129.54" x2="195.58" y2="129.54" width="0.1524" layer="91"/>
+<label x="195.58" y="129.54" size="1.27" layer="95" xref="yes"/>
 </segment>
 </net>
@@
 <pinref part="U$14" gate="G$1" pin="SER"/>
 <wire x1="165.1" y1="170.18" x2="195.58" y2="170.18" width="0.1524" layer="91"/>
+<label x="195.58" y="170.18" size="1.27" layer="95" xref="yes"/>
 </segment>
 </net>
@@
 <pinref part="U$13" gate="G$1" pin="SER"/>
 <wire x1="165.1" y1="210.82" x2="195.58" y2="210.82" width="0.1524" layer="91"/>
+<label x="195.58" y="210.82" size="1.27" layer="95" xref="yes"/>
 </segment>
 </net>
@@
 <pinref part="U$12" gate="G$1" pin="SER"/>
 <wire x1="165.1" y1="254" x2="195.58" y2="254" width="0.1524" layer="91"/>
+<label x="195.58" y="254" size="1.27" layer="95" xref="yes"/>
 </segment>
 </net>
@@
 <pinref part="U$11" gate="G$1" pin="SER"/>
 <wire x1="165.1" y1="294.64" x2="195.58" y2="294.64" width="0.1524" layer="91"/>
+<label x="195.58" y="294.64" size="1.27" layer="95" xref="yes"/>
 </segment>
 </net>
@@
 <pinref part="U$10" gate="G$1" pin="SER"/>
 <wire x1="165.1" y1="335.28" x2="195.58" y2="335.28" width="0.1524" layer="91"/>
+<label x="195.58" y="335.28" size="1.27" layer="95" xref="yes"/>
 </segment>
 </net>
@@
 <pinref part="U$9" gate="G$1" pin="SER"/>
 <wire x1="165.1" y1="375.92" x2="195.58" y2="375.92" width="0.1524" layer="91"/>
+<label x="195.58" y="375.92" size="1.27" layer="95" xref="yes"/>
 </segment>
 </net>
@@
 <pinref part="U$17" gate="G$1" pin="SER"/>
 <wire x1="254" y1="375.92" x2="284.48" y2="375.92" width="0.1524" layer="91"/>
+<label x="284.48" y="375.92" size="1.27" layer="95" xref="yes"/>
 </segment>
 </net>
@@
 <pinref part="U$18" gate="G$1" pin="SER"/>
 <wire x1="254" y1="335.28" x2="284.48" y2="335.28" width="0.1524" layer="91"/>
+<label x="284.48" y="335.28" size="1.27" layer="95" xref="yes"/>
 </segment>
 </net>
@@
 <pinref part="U$19" gate="G$1" pin="SER"/>
 <wire x1="254" y1="294.64" x2="284.48" y2="294.64" width="0.1524" layer="91"/>
+<label x="284.48" y="294.64" size="1.27" layer="95" xref="yes"/>
 </segment>
 </net>
@@
 <pinref part="U$20" gate="G$1" pin="SER"/>
 <wire x1="254" y1="254" x2="284.48" y2="254" width="0.1524" layer="91"/>
+<label x="284.48" y="254" size="1.27" layer="95" xref="yes"/>
 </segment>
 </net>
@@
 <pinref part="U$21" gate="G$1" pin="SER"/>
 <wire x1="254" y1="210.82" x2="284.48" y2="210.82" width="0.1524" layer="91"/>
+<label x="284.48" y="210.82" size="1.27" layer="95" xref="yes"/>
 </segment>
 </net>
@@
 <pinref part="U$22" gate="G$1" pin="SER"/>
 <wire x1="254" y1="170.18" x2="284.48" y2="170.18" width="0.1524" layer="91"/>
+<label x="284.48" y="170.18" size="1.27" layer="95" xref="yes"/>
 </segment>
 </net>
@@
 <pinref part="U$23" gate="G$1" pin="SER"/>
 <wire x1="254" y1="129.54" x2="287.02" y2="129.54" width="0.1524" layer="91"/>
-</segment>
-</net>
+<label x="287.02" y="129.54" size="1.27" layer="95" xref="yes"/>
+</segment>
+</net>
+<net name="N$165" class="0">
+<segment>
+<pinref part="U$6" gate="G$1" pin="SER"/>
+<wire x1="76.2" y1="170.18" x2="106.68" y2="170.18" width="0.1524" layer="91"/>
+<label x="106.68" y="170.18" size="1.27" layer="95" xref="yes"/>
+</segment>
+</net>

Commit message: Adding Stamp board schematic and board layout. Updated SR name labels and updated LED array.
Other:
- moved on the sheet: LED6
Changed lines of the file:
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@@
 </classes>
 <parts>
-<part name="U$1" library="ECE477_Guitutar" deviceset="MM74HC595" device="TSSOP-LD16"/>
 <part name="FRAME1" library="frames" deviceset="FRAME_C_L" device=""/>
 <part name="LED1" library="led" deviceset="LED" device="SMT1206"/>
@@
 <part name="GND23" library="supply1" deviceset="GND" device=""/>
 <part name="P+23" library="supply1" deviceset="VCC" device=""/>
+<part name="U$1" library="ECE477_Guitutar" deviceset="MM74HC595" device="TSSOP-LD16"/>
 </parts>
 <sheets>
@@
 </plain>
 <instances>
-<instance part="U$1" gate="G$1" x="63.5" y="370.84"/>
 <instance part="FRAME1" gate="G$1" x="0" y="0"/>
 <instance part="FRAME1" gate="G$2" x="452.12" y="0"/>
@@
 <instance part="LED4" gate="G$1" x="35.56" y="363.22" rot="R270"/>
 <instance part="LED5" gate="G$1" x="35.56" y="393.7" rot="R270"/>
-<instance part="LED6" gate="G$1" x="81.28" y="378.46" rot="R90"/>
+<instance part="LED6" gate="G$1" x="35.56" y="401.32" rot="R270"/>
 <instance part="GND1" gate="1" x="48.26" y="358.14"/>
 <instance part="P+1" gate="VCC" x="78.74" y="388.62"/>
@@
 <instance part="GND23" gate="1" x="226.06" y="111.76"/>
 <instance part="P+23" gate="VCC" x="256.54" y="142.24"/>
+<instance part="U$1" gate="G$1" x="63.5" y="370.84"/>
 </instances>
 <busses>
@@
 <wire x1="38.1" y1="393.7" x2="47.752" y2="393.7" width="0.1524" layer="91"/>
 <wire x1="47.752" y1="393.7" x2="47.752" y2="381" width="0.1524" layer="91"/>
+<wire x1="47.752" y1="381" x2="50.8" y2="381" width="0.1524" layer="91"/>
 <pinref part="U$1" gate="G$1" pin="QB"/>
-<wire x1="47.752" y1="381" x2="50.8" y2="381" width="0.1524" layer="91"/>
 </segment>
 </net>
@@
 <wire x1="38.1" y1="386.08" x2="42.672" y2="386.08" width="0.1524" layer="91"/>
 <wire x1="42.672" y1="386.08" x2="42.672" y2="378.46" width="0.1524" layer="91"/>
+<wire x1="42.672" y1="378.46" x2="50.8" y2="378.46" width="0.1524" layer="91"/>
 <pinref part="U$1" gate="G$1" pin="QC"/>
-<wire x1="42.672" y1="378.46" x2="50.8" y2="378.46" width="0.1524" layer="91"/>
 </segment>
 </net>
@@
 <wire x1="38.1" y1="378.46" x2="40.132" y2="378.46" width="0.1524" layer="91"/>
 <wire x1="40.132" y1="378.46" x2="40.132" y2="375.92" width="0.1524" layer="91"/>
+<wire x1="40.132" y1="375.92" x2="50.8" y2="375.92" width="0.1524" layer="91"/>
 <pinref part="U$1" gate="G$1" pin="QD"/>
-<wire x1="40.132" y1="375.92" x2="50.8" y2="375.92" width="0.1524" layer="91"/>
 </segment>
 </net>
@@
 <wire x1="38.1" y1="370.84" x2="40.386" y2="370.84" width="0.1524" layer="91"/>
 <wire x1="40.386" y1="370.84" x2="40.386" y2="373.38" width="0.1524" layer="91"/>
+<wire x1="40.386" y1="373.38" x2="50.8" y2="373.38" width="0.1524" layer="91"/>
 <pinref part="U$1" gate="G$1" pin="QE"/>
-<wire x1="40.386" y1="373.38" x2="50.8" y2="373.38" width="0.1524" layer="91"/>
 </segment>
 </net>
@@
 <wire x1="38.1" y1="363.22" x2="43.18" y2="363.22" width="0.1524" layer="91"/>
 <wire x1="43.18" y1="363.22" x2="43.18" y2="370.84" width="0.1524" layer="91"/>
+<wire x1="43.18" y1="370.84" x2="50.8" y2="370.84" width="0.1524" layer="91"/>
 <pinref part="U$1" gate="G$1" pin="QF"/>
-<wire x1="43.18" y1="370.84" x2="50.8" y2="370.84" width="0.1524" layer="91"/>
-</segment>
-</net>
-<net name="N$6" class="0">
-<segment>
-<pinref part="LED6" gate="G$1" pin="A"/>
-<pinref part="U$1" gate="G$1" pin="QA"/>
-<wire x1="78.74" y1="378.46" x2="76.2" y2="378.46" width="0.1524" layer="91"/>
 </segment>
 </net>
@@
 <pinref part="GND1" gate="1" pin="GND"/>
 <wire x1="48.26" y1="360.68" x2="48.26" y2="363.22" width="0.1524" layer="91"/>
+<wire x1="48.26" y1="363.22" x2="50.8" y2="363.22" width="0.1524" layer="91"/>
 <pinref part="U$1" gate="G$1" pin="GND"/>
-<wire x1="48.26" y1="363.22" x2="50.8" y2="363.22" width="0.1524" layer="91"/>
 </segment>
 <segment>
@@
 <net name="VCC" class="0">
 <segment>
-<pinref part="U$1" gate="G$1" pin="VCC"/>
 <wire x1="76.2" y1="381" x2="78.74" y2="381" width="0.1524" layer="91"/>
 <pinref part="P+1" gate="VCC" pin="VCC"/>
 <wire x1="78.74" y1="381" x2="78.74" y2="386.08" width="0.1524" layer="91"/>
+<pinref part="U$1" gate="G$1" pin="VCC"/>
 </segment>
 <segment>
@@
 <net name="N$14" class="0">
 <segment>
-<pinref part="U$1" gate="G$1" pin="G"/>
 <wire x1="76.2" y1="373.38" x2="96.52" y2="373.38" width="0.1524" layer="91"/>
 <wire x1="96.52" y1="373.38" x2="96.52" y2="332.74" width="0.1524" layer="91"/>
@@
 <wire x1="274.32" y1="58.42" x2="302.26" y2="58.42" width="0.1524" layer="91"/>
 <label x="302.26" y="58.42" size="1.27" layer="95" xref="yes"/>
+<pinref part="U$1" gate="G$1" pin="G"/>
 </segment>
 </net>
 <net name="N$16" class="0">
 <segment>
-<pinref part="U$1" gate="G$1" pin="SCK"/>
 <wire x1="76.2" y1="368.3" x2="91.44" y2="368.3" width="0.1524" layer="91"/>
 <wire x1="91.44" y1="368.3" x2="91.44" y2="327.66" width="0.1524" layer="91"/>
@@
 <wire x1="269.24" y1="53.34" x2="292.1" y2="53.34" width="0.1524" layer="91"/>
 <label x="292.1" y="53.34" size="1.27" layer="95" xref="yes"/>
+<pinref part="U$1" gate="G$1" pin="SCK"/>
 </segment>
 </net>
 <net name="N$17" class="0">
 <segment>
-<pinref part="U$1" gate="G$1" pin="SCLR"/>
 <wire x1="76.2" y1="365.76" x2="88.9" y2="365.76" width="0.1524" layer="91"/>
 <wire x1="88.9" y1="365.76" x2="88.9" y2="325.12" width="0.1524" layer="91"/>
@@
 <wire x1="266.7" y1="50.8" x2="287.02" y2="50.8" width="0.1524" layer="91"/>
 <label x="287.02" y="50.8" size="1.27" layer="95" xref="yes"/>
+<pinref part="U$1" gate="G$1" pin="SCLR"/>
 </segment>
 </net>
@@
 <wire x1="182.88" y1="165.1" x2="182.88" y2="124.46" width="0.1524" layer="91"/>
 <wire x1="182.88" y1="248.92" x2="182.88" y2="205.74" width="0.1524" layer="91"/>
-<pinref part="U$1" gate="G$1" pin="RCK"/>
 <wire x1="76.2" y1="370.84" x2="93.98" y2="370.84" width="0.1524" layer="91"/>
 <wire x1="93.98" y1="370.84" x2="93.98" y2="330.2" width="0.1524" layer="91"/>
@@
 <wire x1="271.78" y1="55.88" x2="297.18" y2="55.88" width="0.1524" layer="91"/>
 <label x="297.18" y="55.88" size="1.27" layer="95" xref="yes"/>
+<pinref part="U$1" gate="G$1" pin="RCK"/>
 </segment>
 </net>
 <net name="N$9" class="0">
 <segment>
-<pinref part="U$1" gate="G$1" pin="SER"/>
 <wire x1="76.2" y1="375.92" x2="106.68" y2="375.92" width="0.1524" layer="91"/>
 <label x="106.68" y="375.92" size="1.27" layer="95" xref="yes"/>
+<pinref part="U$1" gate="G$1" pin="SER"/>
 </segment>
 </net>
@@
 </segment>
 </net>
+<net name="N$6" class="0">
+<segment>
+<pinref part="U$1" gate="G$1" pin="QA"/>
+<wire x1="76.2" y1="378.46" x2="81.28" y2="378.46" width="0.1524" layer="91"/>
+<wire x1="81.28" y1="378.46" x2="81.28" y2="401.32" width="0.1524" layer="91"/>
+<pinref part="LED6" gate="G$1" pin="A"/>
+<wire x1="81.28" y1="401.32" x2="38.1" y2="401.32" width="0.1524" layer="91"/>
+</segment>
+</net>
