File: PCB3.sch (EAGLE design)
At the start: 312 parts, among them SW1 CT10-XXXX-A2, SW10 CT10-XXXX-A2, SW100 CT10-XXXX-A2, SW101 CT10-XXXX-A2, SW102 CT10-XXXX-A2, SW103 CT10-XXXX-A2, SW104 CT10-XXXX-A2, SW105 CT10-XXXX-A2, SW106 CT10-XXXX-A2, SW107 CT10-XXXX-A2, SW108 CT10-XXXX-A2, SW109 CT10-XXXX-A2, SW11 CT10-XXXX-A2, SW110 CT10-XXXX-A2, SW111 CT10-XXXX-A2, SW112 CT10-XXXX-A2, SW113 CT10-XXXX-A2, SW114 CT10-XXXX-A2, SW115 CT10-XXXX-A2, SW116 CT10-XXXX-A2, SW117 CT10-XXXX-A2, SW118 CT10-XXXX-A2, SW119 CT10-XXXX-A2, SW12 CT10-XXXX-A2, SW120 CT10-XXXX-A2, SW121 CT10-XXXX-A2, SW122 CT10-XXXX-A2, SW123 CT10-XXXX-A2, SW124 CT10-XXXX-A2, SW125 CT10-XXXX-A2, SW126 CT10-XXXX-A2, SW127 CT10-XXXX-A2, SW128 CT10-XXXX-A2, SW129 CT10-XXXX-A2, SW13 CT10-XXXX-A2, SW130 CT10-XXXX-A2, SW131 CT10-XXXX-A2, SW132 CT10-XXXX-A2, SW14 CT10-XXXX-A2, SW15 CT10-XXXX-A2, SW16 CT10-XXXX-A2, SW17 CT10-XXXX-A2, SW18 CT10-XXXX-A2, SW19 CT10-XXXX-A2, SW2 CT10-XXXX-A2, SW20 CT10-XXXX-A2, SW21 CT10-XXXX-A2, SW22 CT10-XXXX-A2, SW23 CT10-XXXX-A2, SW24 CT10-XXXX-A2, SW25 CT10-XXXX-A2, SW26 CT10-XXXX-A2, SW27 CT10-XXXX-A2, SW28 CT10-XXXX-A2, SW29 CT10-XXXX-A2, SW3 CT10-XXXX-A2, SW30 CT10-XXXX-A2, SW31 CT10-XXXX-A2, SW32 CT10-XXXX-A2, SW33 CT10-XXXX-A2, SW34 CT10-XXXX-A2, SW35 CT10-XXXX-A2, SW36 CT10-XXXX-A2, SW37 CT10-XXXX-A2, SW38 CT10-XXXX-A2, SW39 CT10-XXXX-A2, SW4 CT10-XXXX-A2, SW40 CT10-XXXX-A2, SW41 CT10-XXXX-A2, SW42 CT10-XXXX-A2, SW43 CT10-XXXX-A2, SW44 CT10-XXXX-A2, SW45 CT10-XXXX-A2, SW46 CT10-XXXX-A2, SW47 CT10-XXXX-A2, SW48 CT10-XXXX-A2, SW49 CT10-XXXX-A2, SW5 CT10-XXXX-A2, SW50 CT10-XXXX-A2, SW51 CT10-XXXX-A2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

Commit message: updated schematic to include oscillator, resistor packages, and split main schematic into the five PCBs that we will need. Also started the PCB3 layout that includes the microcontroller.
Parts:
- removed JP1, JP2, JP3, JP4: (no value), pinhead:PINHD-1X25
- removed LED1, LED10, LED100, LED101, LED102, LED103, LED104, LED105, LED106, LED107, LED108, LED109, LED11, LED110, LED111, LED112, LED113, LED114, LED115, LED116, LED117, LED118, LED119, LED12, LED120, LED121, LED122, LED123, LED124, LED125, LED126, LED127, LED128, LED129, LED13, LED130, LED131, LED132, LED133, LED134, LED135, LED136, LED137, LED138, LED139, LED14, LED15, LED16, LED17, LED18, LED19, LED2, LED20, LED21, LED22, LED23, LED24, LED25, LED26, LED27, LED28, LED29, LED3, LED30, LED31, LED32, LED33, LED34, LED35, LED36, LED37, LED38, LED39, LED4, LED40, LED41, LED42, LED43, LED44, LED45, LED46, LED47, LED48, LED49, LED5, LED50, LED51, LED52, LED53, LED54, LED55, LED56, LED57, LED58, LED59, LED6, LED60, LED61, LED62, LED63, LED64, LED65, LED66, LED67, LED68, LED69, LED7, LED70, LED71, LED72, LED73, LED74, LED75, LED76, LED77, LED78, LED79, LED8, LED80, LED81, LED82, LED83, LED84, LED85, LED86, LED87, LED88, LED89, LED9, LED90, LED91, LED92, LED93, LED94, LED95, LED96, LED97, LED98, LED99: (no value), led:LEDSMT1206
- removed SW1, SW10, SW100, SW101, SW102, SW103, SW104, SW105, SW106, SW107, SW108, SW109, SW11, SW110, SW111, SW112, SW113, SW114, SW115, SW116, SW117, SW118, SW119, SW12, SW120, SW121, SW122, SW123, SW124, SW125, SW126, SW127, SW128, SW129, SW13, SW130, SW131, SW132, SW14, SW15, SW16, SW17, SW18, SW19, SW2, SW20, SW21, SW22, SW23, SW24, SW25, SW26, SW27, SW28, SW29, SW3, SW30, SW31, SW32, SW33, SW34, SW35, SW36, SW37, SW38, SW39, SW4, SW40, SW41, SW42, SW43, SW44, SW45, SW46, SW47, SW48, SW49, SW5, SW50, SW51, SW52, SW53, SW54, SW55, SW56, SW57, SW58, SW59, SW6, SW60, SW61, SW62, SW63, SW64, SW65, SW66, SW67, SW68, SW69, SW7, SW70, SW71, SW72, SW73, SW74, SW75, SW76, SW77, SW78, SW79, SW8, SW80, SW81, SW82, SW83, SW84, SW85, SW86, SW87, SW88, SW89, SW9, SW90, SW91, SW92, SW93, SW94, SW95, SW96, SW97, SW98, SW99: CT10-XXXX-A2, switch-coto:CT10-XXXX-A2
- removed U$10, U$11, U$12, U$13, U$14, U$15, U$16, U$17, U$18, U$19, U$20, U$21, U$22, U$23, U$24, U$25, U$3, U$4, U$5, U$6, U$7, U$8, U$9: MM74HC595TSSOP-LD16, ECE477_Guitutar:MM74HC595TSSOP-LD16
- removed U$2: BM78SPP05MC2/NC2, ECE477_Guitutar:BM78SPP05MC2/NC2
- added C9: (no value), rcl:C-USC0805
- added LED140, LED141, LED142, LED143, LED144, LED145, LED146, LED147, LED148, LED149, LED150, LED151, LED152, LED153, LED154, LED155, LED156, LED157, LED158, LED159, LED160, LED161, LED162, LED163: (no value), led:LEDSMT1206
- added R4, R5, R6, R7: (no value), resistor-bourns:4814P-T01
- added R8: (no value), rcl:R-US_M0805
- added U$26, U$27, U$28, U$29: MM74HC595TSSOP-LD16, ECE477_Guitutar:MM74HC595TSSOP-LD16
- added Y1: (no value), SparkFun-Clocks:CRYSTALSMD-5X3.2-2PAD
Connections:
- removed net EAN: U$2.EAN
- removed net FRET16: JP3.13, SW91.2, SW92.2, SW93.2, SW94.2, SW95.2, SW96.2, U$1.OSC1/CLKI/RC12
- removed net FRET17: JP3.14, SW100.2, SW101.2, SW102.2, SW97.2, SW98.2, SW99.2, U$1.OSC2/CLKO/RC15
- removed net LED: LED1.C, U$2.LED1
- removed net N$107: LED34.A, U$8.QD
- removed net N$108: LED35.A, U$8.QE
- removed net N$109: LED33.A, U$8.QC
- removed net N$11: LED5.A, U$3.QE
- removed net N$110: LED32.A, U$8.QB
- removed net N$111: LED36.A, U$8.QF
- removed net N$117: LED37.A, U$8.QA
- removed net N$118: LED40.A, U$9.QD
- removed net N$119: LED41.A, U$9.QE
- removed net N$120: LED39.A, U$9.QC
- removed net N$121: LED38.A, U$9.QB
- removed net N$122: LED42.A, U$9.QF
- removed net N$128: LED43.A, U$9.QA
- removed net N$129: LED46.A, U$10.QD
- removed net N$130: LED47.A, U$10.QE
- removed net N$131: LED45.A, U$10.QC
- removed net N$132: LED44.A, U$10.QB
- removed net N$133: LED48.A, U$10.QF
- removed net N$139: LED49.A, U$10.QA
- removed net N$140: LED52.A, U$11.QD
- removed net N$141: LED53.A, U$11.QE
- removed net N$142: LED51.A, U$11.QC
- removed net N$143: LED50.A, U$11.QB
- removed net N$144: LED54.A, U$11.QF
- removed net N$15: LED1.A, R3.1
- removed net N$150: LED55.A, U$11.QA
- removed net N$151: LED58.A, U$12.QD
- removed net N$152: LED59.A, U$12.QE
- removed net N$153: LED57.A, U$12.QC
- removed net N$154: LED56.A, U$12.QB
- removed net N$155: LED60.A, U$12.QF
- removed net N$16: R3.2, U$2.LDO33_O, U$2.VDD_IO
- removed net N$161: LED61.A, U$12.QA
- removed net N$162: LED64.A, U$13.QD
- removed net N$163: LED65.A, U$13.QE
- removed net N$164: LED63.A, U$13.QC
- removed net N$165: LED62.A, U$13.QB
- removed net N$166: LED66.A, U$13.QF
- removed net N$17: LED3.A, U$3.QC
- removed net N$172: LED67.A, U$13.QA
- removed net N$173: LED70.A, U$14.QD
- removed net N$174: LED71.A, U$14.QE
- removed net N$175: LED69.A, U$14.QC
- removed net N$176: LED68.A, U$14.QB
- removed net N$177: LED72.A, U$14.QF
- removed net N$18: LED2.A, U$3.QB
- removed net N$183: LED73.A, U$14.QA
- removed net N$184: LED76.A, U$15.QD
- removed net N$185: LED77.A, U$15.QE
- removed net N$186: LED75.A, U$15.QC
- removed net N$187: LED74.A, U$15.QB
- removed net N$188: LED78.A, U$15.QF
- removed net N$19: LED6.A, U$3.QF
- removed net N$194: LED79.A, U$15.QA
- removed net N$195: LED82.A, U$16.QD
- removed net N$196: LED83.A, U$16.QE
- removed net N$197: LED81.A, U$16.QC
- removed net N$198: LED80.A, U$16.QB
- removed net N$199: LED84.A, U$16.QF
- removed net N$205: LED85.A, U$16.QA
- removed net N$206: LED88.A, U$17.QD
- removed net N$207: LED89.A, U$17.QE
- removed net N$208: LED87.A, U$17.QC
- removed net N$209: LED86.A, U$17.QB
- removed net N$210: LED90.A, U$17.QF
- removed net N$216: LED91.A, U$17.QA
- removed net N$217: LED94.A, U$18.QD
- removed net N$218: LED95.A, U$18.QE
- removed net N$219: LED93.A, U$18.QC
- removed net N$220: LED92.A, U$18.QB
- removed net N$221: LED96.A, U$18.QF
- removed net N$227: LED97.A, U$18.QA
- removed net N$228: LED100.A, U$19.QD
- removed net N$229: LED101.A, U$19.QE
- removed net N$230: LED99.A, U$19.QC
- removed net N$231: LED98.A, U$19.QB
- removed net N$232: LED102.A, U$19.QF
- removed net N$238: LED103.A, U$19.QA
- removed net N$239: LED106.A, U$20.QD
- removed net N$240: LED107.A, U$20.QE
- removed net N$241: LED105.A, U$20.QC
- removed net N$242: LED104.A, U$20.QB
- removed net N$243: LED108.A, U$20.QF
- removed net N$249: LED109.A, U$20.QA
- removed net N$250: LED112.A, U$21.QD
- removed net N$251: LED113.A, U$21.QE
- removed net N$252: LED111.A, U$21.QC
- removed net N$253: LED110.A, U$21.QB
- removed net N$254: LED114.A, U$21.QF
- removed net N$26: LED10.A, U$4.QD
- removed net N$260: LED115.A, U$21.QA
- removed net N$261: LED118.A, U$22.QD
- removed net N$262: LED119.A, U$22.QE
- removed net N$263: LED117.A, U$22.QC
- removed net N$264: LED116.A, U$22.QB
- removed net N$265: LED120.A, U$22.QF
- removed net N$27: LED11.A, U$4.QE
- removed net N$271: LED121.A, U$22.QA
- removed net N$272: LED124.A, U$23.QD
- removed net N$273: LED125.A, U$23.QE
- removed net N$274: LED123.A, U$23.QC
- removed net N$275: LED122.A, U$23.QB
- removed net N$276: LED126.A, U$23.QF
- removed net N$28: LED9.A, U$4.QC
- removed net N$282: LED127.A, U$23.QA
- removed net N$283: LED130.A, U$24.QD
- removed net N$284: LED131.A, U$24.QE
- removed net N$285: LED129.A, U$24.QC
- removed net N$286: LED128.A, U$24.QB
- removed net N$287: LED132.A, U$24.QF
- removed net N$29: LED8.A, U$4.QB
- removed net N$293: LED133.A, U$24.QA
- removed net N$294: LED136.A, U$25.QD
- removed net N$295: LED137.A, U$25.QE
- removed net N$296: LED135.A, U$25.QC
- removed net N$297: LED134.A, U$25.QB
- removed net N$298: LED138.A, U$25.QF
- removed net N$304: LED139.A, U$25.QA
- removed net N$36: LED13.A, U$4.QA
- removed net N$39: LED15.A, U$5.QC
- removed net N$40: LED14.A, U$5.QB
- removed net N$41: LED18.A, U$5.QF
- removed net N$54: LED19.A, U$5.QA
- removed net N$55: LED22.A, U$6.QD
- removed net N$56: LED23.A, U$6.QE
- removed net N$57: LED21.A, U$6.QC
- removed net N$58: LED20.A, U$6.QB
- removed net N$59: LED24.A, U$6.QF
- removed net N$6: LED7.A, U$3.QA
- removed net N$65: LED25.A, U$6.QA
- removed net N$69: LED28.A, U$7.QD
- removed net N$70: LED29.A, U$7.QE
- removed net N$71: LED27.A, U$7.QC
- removed net N$72: LED26.A, U$7.QB
- removed net N$73: LED30.A, U$7.QF
- removed net N$79: LED31.A, U$7.QA
- removed net N$8: LED4.A, U$3.QD
- removed net P1_2: U$2.P1_2/SCL
- removed net P1_3: U$2.P1_3/SDA
- removed net P2_0: U$2.P2_0
- removed net P2_4: U$2.P2_4
- removed net P3_6: U$2.P3_6
- removed net VCC: U$10.VCC, U$11.VCC, U$12.VCC, U$13.VCC, U$14.VCC, U$15.VCC, U$16.VCC, U$17.VCC, U$18.VCC, U$19.VCC, U$20.VCC, U$21.VCC, U$22.VCC, U$23.VCC, U$24.VCC, U$25.VCC, U$3.VCC, U$4.VCC, U$5.VCC, U$6.VCC, U$7.VCC, U$8.VCC, U$9.VCC
- new net N$100: LED156.A, R6.5
- new net N$101: LED157.A, R6.6
- new net N$102: LED153.A, R6.2
- new net N$103: U$29.SER
- new net N$113: R7.13, U$26.QB
- new net N$114: R7.12, U$26.QC
- new net N$115: R7.11, U$26.QD
- new net N$116: R7.10, U$26.QE
- new net N$123: R7.9, U$26.QF
- new net N$124: U$26.VCC
- new net N$125: R7.14, U$26.QA
- new net N$126: LED158.A, R7.1
- new net N$127: LED160.A, R7.3
- new net N$134: LED161.A, R7.4
- new net N$135: LED162.A, R7.5
- new net N$136: LED163.A, R7.6
- new net N$137: LED159.A, R7.2
- new net N$138: U$26.SER
- new net N$20: R4.13, U$27.QB
- new net N$21: R4.12, U$27.QC
- new net N$22: R4.11, U$27.QD
- new net N$23: R4.10, U$27.QE
- new net N$24: R4.9, U$27.QF
- new net N$25: U$27.VCC
- new net N$31: R4.14, U$27.QA
- new net N$32: LED140.A, R4.1
- new net N$33: LED141.A, R4.2
- new net N$34: LED142.A, R4.3
- new net N$35: LED143.A, R4.4
- new net N$46: LED144.A, R4.5
- new net N$47: LED145.A, R4.6
- new net N$48: U$27.SER
- new net N$62: R5.13, U$28.QB
- new net N$63: R5.12, U$28.QC
- new net N$64: R5.11, U$28.QD
- new net N$74: R5.10, U$28.QE
- new net N$75: R5.9, U$28.QF
- new net N$76: U$28.VCC
- new net N$77: R5.14, U$28.QA
- new net N$78: LED146.A, R5.1
- new net N$80: LED148.A, R5.3
- new net N$81: LED149.A, R5.4
- new net N$82: LED150.A, R5.5
- new net N$83: LED151.A, R5.6
- new net N$84: LED147.A, R5.2
- new net N$85: U$28.SER
- new net N$90: R6.13, U$29.QB
- new net N$91: R6.12, U$29.QC
- new net N$92: R6.11, U$29.QD
- new net N$93: R6.10, U$29.QE
- new net N$94: R6.9, U$29.QF
- new net N$95: U$29.VCC
- new net N$96: R6.14, U$29.QA
- new net N$97: LED152.A, R6.1
- new net N$98: LED154.A, R6.3
- new net N$99: LED155.A, R6.4
- net FRET1: no longer JP2.16, SW1.2, SW2.2, SW3.2, SW4.2, SW5.2, SW6.2
- net FRET10: no longer JP3.2, SW55.2, SW56.2, SW57.2, SW58.2, SW59.2, SW60.2
- net FRET11: no longer JP3.3, SW61.2, SW62.2, SW63.2, SW64.2, SW65.2, SW66.2
- net FRET12: no longer JP3.8, SW67.2, SW68.2, SW69.2, SW70.2, SW71.2, SW72.2
- net FRET13: no longer JP3.9, SW73.2, SW74.2, SW75.2, SW76.2, SW77.2, SW78.2
- net FRET14: no longer JP3.10, SW79.2, SW80.2, SW81.2, SW82.2, SW83.2, SW84.2
- net FRET15: no longer JP3.11, SW85.2, SW86.2, SW87.2, SW88.2, SW89.2, SW90.2
- net FRET18: no longer JP3.16, SW103.2, SW104.2, SW105.2, SW106.2, SW107.2, SW108.2
- net FRET19: no longer JP3.17, SW109.2, SW110.2, SW111.2, SW112.2, SW113.2, SW114.2
- net FRET2: no longer JP2.17, SW10.2, SW11.2, SW12.2, SW7.2, SW8.2, SW9.2
- net FRET20: no longer JP3.18, SW115.2, SW116.2, SW117.2, SW118.2, SW119.2, SW120.2
- net FRET21: no longer JP3.19, SW121.2, SW122.2, SW123.2, SW124.2, SW125.2, SW126.2
- net FRET22: no longer JP3.20, SW127.2, SW128.2, SW129.2, SW130.2, SW131.2, SW132.2
- net FRET3: no longer JP2.18, SW13.2, SW14.2, SW15.2, SW16.2, SW17.2, SW18.2
- net FRET4: no longer JP2.19, SW19.2, SW20.2, SW21.2, SW22.2, SW23.2, SW24.2
- net FRET5: no longer JP2.22, SW25.2, SW26.2, SW27.2, SW28.2, SW29.2, SW30.2
- net FRET6: no longer JP2.23, SW31.2, SW32.2, SW33.2, SW34.2, SW35.2, SW36.2
- net FRET7: no longer JP2.24, SW37.2, SW38.2, SW39.2, SW40.2, SW41.2, SW42.2
- net FRET8: no longer JP2.25, SW43.2, SW44.2, SW45.2, SW46.2, SW47.2, SW48.2
- net FRET9: no longer JP3.1, SW49.2, SW50.2, SW51.2, SW52.2, SW53.2, SW54.2
- net G: now also U$26.G, U$27.G, U$28.G, U$29.G; no longer JP3.24, U$10.G, U$11.G, U$12.G, U$13.G, U$14.G, U$15.G, U$16.G, U$17.G, U$18.G, U$19.G, U$20.G, U$21.G, U$22.G, U$23.G, U$24.G, U$25.G, U$3.G, U$4.G, U$5.G, U$6.G, U$7.G, U$8.G, U$9.G
- net GND: now also C8.1, C9.2, U$26.GND, U$27.GND, U$28.GND, U$29.GND; no longer LED10.C, LED100.C, LED101.C, LED102.C, LED103.C, LED104.C, LED105.C, LED106.C, LED107.C, LED108.C, LED109.C, LED11.C, LED110.C, LED111.C, LED112.C, LED113.C, LED114.C, LED115.C, LED116.C, LED117.C, LED118.C, LED119.C, LED12.C, LED120.C, LED121.C, LED122.C, LED123.C, LED124.C, LED125.C, LED126.C, LED127.C, LED128.C, LED129.C, LED13.C, LED130.C, LED131.C, LED132.C, LED133.C, LED134.C, LED135.C, LED136.C, LED137.C, LED138.C, LED139.C, LED14.C, LED15.C, LED16.C, LED17.C, LED18.C, LED19.C, LED2.C, LED20.C, LED21.C, LED22.C, LED23.C, LED24.C, LED25.C, LED26.C, LED27.C, LED28.C, LED29.C, LED3.C, LED30.C, LED31.C, LED32.C, LED33.C, LED34.C, LED35.C, LED36.C, LED37.C, LED38.C, LED39.C, LED4.C, LED40.C, LED41.C, LED42.C, LED43.C, LED44.C, LED45.C, LED46.C, LED47.C, LED48.C, LED49.C, LED5.C, LED50.C, LED51.C, LED52.C, LED53.C, LED54.C, LED55.C, LED56.C, LED57.C, LED58.C, LED59.C, LED6.C, LED60.C, LED61.C, LED62.C, LED63.C, LED64.C, LED65.C, LED66.C, LED67.C, LED68.C, LED69.C, LED7.C, LED70.C, LED71.C, LED72.C, LED73.C, LED74.C, LED75.C, LED76.C, LED77.C, LED78.C, LED79.C, LED8.C, LED80.C, LED81.C, LED82.C, LED83.C, LED84.C, LED85.C, LED86.C, LED87.C, LED88.C, LED89.C, LED9.C, LED90.C, LED91.C, LED92.C, LED93.C, LED94.C, LED95.C, LED96.C, LED97.C, LED98.C, LED99.C, U$10.GND, U$11.GND, U$12.GND, U$13.GND, U$14.GND, U$15.GND, U$16.GND, U$17.GND, U$18.GND, U$19.GND, U$20.GND, U$21.GND, U$22.GND, U$23.GND, U$24.GND, U$25.GND, U$3.GND, U$4.GND, U$5.GND, U$6.GND, U$7.GND, U$8.GND, U$9.GND
- net LED_SER1: no longer JP4.25, U$3.SER
- net LED_SER10: no longer JP4.16, U$12.SER
- net LED_SER11: no longer JP4.15, U$13.SER
- net LED_SER12: no longer JP4.14, U$14.SER
- net LED_SER13: no longer JP4.13, U$15.SER
- net LED_SER14: no longer JP4.12, U$16.SER
- net LED_SER15: no longer JP4.9, U$17.SER
- net LED_SER16: no longer JP4.8, U$18.SER
- net LED_SER17: no longer JP4.7, U$19.SER
- net LED_SER18: no longer JP4.6, U$20.SER
- net LED_SER19: no longer JP4.5, U$21.SER
- net LED_SER2: no longer JP4.24, U$4.SER
- net LED_SER20: no longer JP4.4, U$22.SER
- net LED_SER21: no longer JP4.3, U$23.SER
- net LED_SER22: no longer JP4.2, U$24.SER
- net LED_SER23: no longer JP4.1, U$25.SER
- net LED_SER3: no longer JP4.23, U$5.SER
- net LED_SER4: no longer JP4.22, U$6.SER
- net LED_SER5: no longer JP4.21, U$7.SER
- net LED_SER6: no longer JP4.20, U$8.SER
- net LED_SER7: no longer JP4.19, U$9.SER
- net LED_SER8: no longer JP4.18, U$10.SER
- net LED_SER9: no longer JP4.17, U$11.SER
- net N$10: no longer JP4.11
- net N$12: no longer JP4.10
- net N$13: no longer JP1.13
- net N$14: no longer JP1.25
- net N$2: no longer JP1.24
- net N$3: no longer JP1.17
- net N$30: now also R3.2, R8.1, U$1.OSC2/CLKO/RC15; no longer LED12.A, U$4.QF
- net N$37: now also C9.1, R3.1, Y1.2; no longer LED16.A, U$5.QD
- net N$38: now also C8.2, R8.2, U$1.OSC1/CLKI/RC12, Y1.1; no longer LED17.A, U$5.QE
- net N$4: no longer JP1.22
- net N$42: no longer JP2.1
- net N$43: no longer JP2.2
- net N$44: no longer JP2.3
- net N$45: no longer JP2.4
- net N$5: no longer JP1.23
- net N$50: no longer JP2.11
- net N$51: no longer JP2.12
- net N$52: no longer JP2.13
- net N$66: no longer JP3.4
- net N$67: no longer JP3.6
- net N$68: no longer JP3.7
- net N$7: no longer JP2.21
- net N$9: no longer JP3.12, JP3.5
- net P0_0: no longer JP1.14, JP1.18, U$2.P0_0
- net P0_4: no longer JP1.3, U$2.P0_4
- net P0_5: no longer JP1.12, U$2.P0_5
- net P1_5: no longer JP1.1, U$2.P1_5
- net P1_7: no longer JP1.19, U$2.P1_7
- net P3_1: no longer JP1.11, U$2.P3_1
- net P3_2: no longer JP1.10, U$2.P3_2
- net P3_3: no longer JP1.9, U$2.P3_3
- net P3_4: no longer JP1.8, U$2.P3_4
- net P3_7: no longer JP1.7, U$2.P3_7
- net PE: no longer C8.2, U$2.GND, U$2.GND1
- net RCK: now also U$26.RCK, U$27.RCK, U$28.RCK, U$29.RCK; no longer JP3.23, U$10.RCK, U$11.RCK, U$12.RCK, U$13.RCK, U$14.RCK, U$15.RCK, U$16.RCK, U$17.RCK, U$18.RCK, U$19.RCK, U$20.RCK, U$21.RCK, U$22.RCK, U$23.RCK, U$24.RCK, U$25.RCK, U$3.RCK, U$4.RCK, U$5.RCK, U$6.RCK, U$7.RCK, U$8.RCK, U$9.RCK
- net RST_N: no longer JP1.6, U$2.RST_N
- net RXD: no longer JP1.21, U$2.HCI_RXD
- net SCK: now also U$26.SCK, U$27.SCK, U$28.SCK, U$29.SCK; no longer JP3.22, U$10.SCK, U$11.SCK, U$12.SCK, U$13.SCK, U$14.SCK, U$15.SCK, U$16.SCK, U$17.SCK, U$18.SCK, U$19.SCK, U$20.SCK, U$21.SCK, U$22.SCK, U$23.SCK, U$24.SCK, U$25.SCK, U$3.SCK, U$4.SCK, U$5.SCK, U$6.SCK, U$7.SCK, U$8.SCK, U$9.SCK
- net SCLR: now also U$26.SCLR, U$27.SCLR, U$28.SCLR, U$29.SCLR; no longer JP3.21, U$10.SCLR, U$11.SCLR, U$12.SCLR, U$13.SCLR, U$14.SCLR, U$15.SCLR, U$16.SCLR, U$17.SCLR, U$18.SCLR, U$19.SCLR, U$20.SCLR, U$21.SCLR, U$22.SCLR, U$23.SCLR, U$24.SCLR, U$25.SCLR, U$3.SCLR, U$4.SCLR, U$5.SCLR, U$6.SCLR, U$7.SCLR, U$8.SCLR, U$9.SCLR
- net STRING1: no longer JP2.7, SW1.1, SW102.1, SW108.1, SW114.1, SW12.1, SW120.1, SW126.1, SW132.1, SW18.1, SW24.1, SW30.1, SW36.1, SW42.1, SW48.1, SW54.1, SW60.1, SW66.1, SW72.1, SW78.1, SW84.1, SW90.1, SW96.1
- net STRING2: no longer JP2.8, SW103.1, SW109.1, SW115.1, SW121.1, SW127.1, SW13.1, SW19.1, SW2.1, SW25.1, SW31.1, SW37.1, SW43.1, SW49.1, SW55.1, SW61.1, SW67.1, SW7.1, SW73.1, SW79.1, SW85.1, SW91.1, SW97.1
- net STRING3: no longer JP2.9, SW104.1, SW110.1, SW116.1, SW122.1, SW128.1, SW14.1, SW20.1, SW26.1, SW3.1, SW32.1, SW38.1, SW44.1, SW50.1, SW56.1, SW62.1, SW68.1, SW74.1, SW8.1, SW80.1, SW86.1, SW92.1, SW98.1
- net STRING4: no longer JP2.10, SW105.1, SW111.1, SW117.1, SW123.1, SW129.1, SW15.1, SW21.1, SW27.1, SW33.1, SW39.1, SW4.1, SW45.1, SW51.1, SW57.1, SW63.1, SW69.1, SW75.1, SW81.1, SW87.1, SW9.1, SW93.1, SW99.1
- net STRING5: no longer JP2.14, SW10.1, SW100.1, SW106.1, SW112.1, SW118.1, SW124.1, SW130.1, SW16.1, SW22.1, SW28.1, SW34.1, SW40.1, SW46.1, SW5.1, SW52.1, SW58.1, SW64.1, SW70.1, SW76.1, SW82.1, SW88.1, SW94.1
- net STRING6: no longer JP2.15, SW101.1, SW107.1, SW11.1, SW113.1, SW119.1, SW125.1, SW131.1, SW17.1, SW23.1, SW29.1, SW35.1, SW41.1, SW47.1, SW53.1, SW59.1, SW6.1, SW65.1, SW71.1, SW77.1, SW83.1, SW89.1, SW95.1
- net SW_BTN: no longer JP1.4, U$2.SW_BTN
- net TXD: no longer JP1.20, U$2.HCI_TXD
- net VDD: no longer C8.1, JP1.16, JP1.2, JP2.5, U$2.BAT_IN
- net VSS: no longer JP1.15, JP2.20, JP2.6, JP3.15, JP3.25
- net WAKEUP: no longer JP1.5, U$2.WAKEUP
