File: PCB1.brd (EAGLE design)
At the start: 101.4 x 47.5 mm, 71 parts

Commit message: Finished changing dimensions for PCB3 and switched out resistors for smaller ones.
Connections:
- net N$14 renamed SCLR
- net N$48 renamed SCK
- net N$51 renamed RCK
Changed lines of the file:
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@@
 <?xml version="1.0" encoding="utf-8"?>
 <!DOCTYPE eagle SYSTEM "eagle.dtd">
-<eagle version="8.1.0">
+<eagle version="8.0.1">
 <drawing>
 <settings>
@@
 <wire x1="86.614" y1="16.51" x2="90.17" y2="20.066" width="0.254" layer="1"/>
 </signal>
-<signal name="N$48">
+<signal name="SCK">
 <contactref element="U$4" pad="11"/>
 <contactref element="U$1" pad="11"/>
@@
 <wire x1="77.724" y1="9.906" x2="78.486" y2="9.906" width="0" layer="19" extent="1-16"/>
 </signal>
-<signal name="N$51">
+<signal name="RCK">
 <contactref element="U$4" pad="12"/>
 <contactref element="U$1" pad="12"/>
@@
 <wire x1="92.202" y1="11.938" x2="90.976" y2="11.938" width="0.254" layer="16"/>
 </signal>
-<signal name="N$14">
+<signal name="SCLR">
 <contactref element="U$4" pad="10"/>
 <contactref element="U$1" pad="10"/>
